Commit message: Cámara articulable

File: retos_ws/src/articubot_one/description/camera.xacro (robot description, xacro)
@@ -1,17 +1,31 @@
 <?xml version="1.0"?>
 <robot xmlns:xacro="http://www.ros.org/wiki/xacro" >
-    <joint name="camera_joint" type="fixed">
-        <parent link="chassis"/>
+    <xacro:include filename="inertial_macros.xacro"/>
+    <joint name="camera_joint" type="revolute">
+        <parent link="base_link"/>
         <child link="camera_link"/>
-        <origin xyz="0.257 0 0.070" rpy="0 1.57 0"/>
+        <origin xyz="0.205 0 0.08" rpy="0 0 0"/>
+        <axis xyz="0 1 0"/>
+        <limit lower="0" upper="${pi/2}" velocity="100" effort="0.5"/>
     </joint>
     <link name="camera_link">
         <visual>
             <geometry>
-                <box size="0.001 0.03 0.03"/>
+                <box size="0.010 0.03 0.03"/>
             </geometry>
-            <material name="black"/>
+            <material name="red"/>
         </visual>
+        <collision>
+            <geometry>
+                <sphere radius="0.01"/>
+            </geometry>
+        </collision>
+        <xacro:inertial_box mass="0.001" x="0.0001" y="0.0001" z="0.0001">
+            <origin xyz="0 0 0" rpy="0 0 0"/>
+        </xacro:inertial_box>
     </link>
+    <gazebo reference="camera_link">
+        <material>Gazebo/Red</material>
+    </gazebo>
     <joint name="camera_optical_joint" type="fixed">
         <parent link="camera_link"/>
@@ -20,6 +34,19 @@
     </joint>
     <link name="camera_link_optical"></link>
+    <gazebo>
+        <plugin name="gazebo_ros_joint_state_publisher"
+            filename="libgazebo_ros_joint_state_publisher.so">
+            <update_rate>20</update_rate>
+            <joint_name>camera_joint</joint_name>
+        </plugin>
+    </gazebo>
+    <gazebo>
+        <plugin name="gazebo_ros_joint_pose_trajectory"
+            filename="libgazebo_ros_joint_pose_trajectory.so">
+            <update_rate>2</update_rate>
+        </plugin>
+    </gazebo>
     <gazebo reference="camera_link">
-        <material>Gazebo/Black</material>
+        <material>Gazebo/Red</material>
         <sensor name="camera" type="camera">
             <pose> 0 0 0 0 0 0 </pose>
@@ -41,4 +68,11 @@
                 <frame_name>camera_link_optical</frame_name>
             </plugin>
+            <plugin name="gazebo_ros_control" filename="libgazebo_ros_control.so">
+                <robotNamespace>/</robotNamespace>
+            </plugin>
+            <plugin name="camera_control_plugin" filename="libcamera_control_plugin.so">
+                <command_topic>/camera_control</command_topic>
+                <robot_namespace>/</robot_namespace>
+            </plugin>
         </sensor>
     </gazebo>

File: retos_ws/src/articubot_one/description/robot_core.xacro (robot description, xacro)
@@ -3,5 +3,5 @@
     <xacro:include filename="inertial_macros.xacro"/>
     <!-- Define camera tilt angle -->
-    <xacro:property name="camera_tilt_angle" value="0.0"/>
+    <xacro:property name="camera_link_tilt" value="0.0"/>
     <xacro:property name="chassis_length" value="0.225"/>
     <xacro:property name="chassis_width" value="0.160"/>
@@ -70,19 +70,4 @@
             <origin xyz="${chassis_length/2} 0 ${chassis_height/2}" rpy="0 0 0"/>
         </xacro:inertial_box>
-    </link>
-    <!-- Add camera joint for tilting -->
-    <joint name="camera_tilt_joint" type="continuous">
-        <parent link="chassis"/>
-        <child link="camera_tilt_link"/>
-        <origin xyz="0.257 0 0.070" rpy="0 0 ${camera_tilt_angle}"/>
-        <axis xyz="0 0 1"/>
-    </joint>
-    <link name="camera_tilt_link">
-        <visual>
-            <geometry>
-                <box size="0.001 0.03 0.03"/>
-            </geometry>
-            <material name="black"/>
-        </visual>
     </link>
     <!-- LEFT WHEEL LINK -->
@@ -165,3 +150,13 @@
         <mu2 value="0.001"/>
     </gazebo>
+    <gazebo>
+        <plugin filename="libgazebo_ros2_control.so" name="gazebo_ros2_control">
+            <ros>
+                <namespace>/</namespace>
+                <parameter_file_ws>/path_to_workspace</parameter_file_ws>
+            </ros>
+            <robotSimType>gazebo_ros2_control/DefaultRobotHWSim</robotSimType>
+            <robotParam>robot_description</robotParam>
+        </plugin>
+    </gazebo>
 </robot>

Commit message: juankarlos debuelveme mis auriculares

File: retos_ws/src/articubot_one/description/camera.xacro (robot description, xacro)
@@ -5,5 +5,5 @@
         <parent link="base_link"/>
         <child link="camera_link"/>
-        <origin xyz="0.205 0 0.08" rpy="0 0 0"/>
+        <origin xyz="0.205 0 0.08" rpy="0 0 0"/>   <!-- Para cambiar la altura de la cámara, modifica el valor z. Ideal para altura de robot: 0.08. Más altura depende del campo de visión que se necesite -->
         <axis xyz="0 1 0"/>
         <limit lower="0" upper="${pi/2}" velocity="100" effort="0.5"/>
@@ -82,4 +82,5 @@
             <!-- Wheel Information -->
             <left_joint>camera_joint</left_joint>
+            <right_joint>new_joint</right_joint>
             <!-- Limits -->
             <max_wheel_torque>200</max_wheel_torque>
