Commit message: Solucion de los errores del simulador_gazebo

File: retos_ws/src/simulador_gazebo/description/ros2_control.xacro (robot description, xacro)
@@ -56,6 +56,6 @@
     <gazebo>
         <plugin name="gazebo_ros2_control" filename="libgazebo_ros2_control.so">
-            <parameters>$(find articubot_one)/config/my_controllers.yaml</parameters>
-            <parameters>$(find articubot_one)/config/gaz_ros2_ctl_use_sim.yaml</parameters>
+            <parameters>$(find simulador_gazebo)/config/my_controllers.yaml</parameters>
+            <parameters>$(find simulador_gazebo)/config/gaz_ros2_ctl_use_sim.yaml</parameters>
         </plugin>
     </gazebo>

File: retos_ws/src/simulador_gazebo/models/Cybercrex_frontal/camera.xacro (robot description, xacro)
@@ -4,5 +4,5 @@
         <parent link="chassis"/>
         <child link="camera_link"/>
-        <origin xyz="0.257 0 0.46" rpy="0 0.523599 0"/>
+        <origin xyz="0.257 0 1.0" rpy="0 0.523599 0"/>
     </joint>
     <link name="camera_link">

File: retos_ws/src/simulador_gazebo/models/Cybercrex_frontal/robot.urdf.xacro (robot description, xacro)
@@ -1,6 +1,6 @@
 <?xml version="1.0"?>
 <robot xmlns:xacro="http://www.ros.org/wiki/xacro"  name="cybercrex">
-    <xacro:arg name="use_ros2_control" default="true"/>
-    <xacro:arg name="sim_mode" default="false"/>
+    <xacro:arg name="use_ros2_control" default="false"/>
+    <xacro:arg name="sim_mode" default="true"/>
     <xacro:include filename="robot_core.xacro" />
     <xacro:if value="$(arg use_ros2_control)">
