Commit message: Programa de detecion de texto con easyocr

File: retos_ws/src/simulador_gazebo/models/Cybercrex_frontal/camera.xacro (robot description, xacro)
@@ -4,5 +4,5 @@
         <parent link="chassis"/>
         <child link="camera_link"/>
-        <origin xyz="0.257 0 1.0" rpy="0 0.523599 0"/>
+        <origin xyz="0.257 0 1.165" rpy="0 0.523599 0"/>
     </joint>
     <link name="camera_link">
