Commit message: Deteccion de formas completado

File: retos_ws/src/simulador_gazebo/models/Cybercrex_figuras/camera.xacro (robot description, xacro)
@@ -4,5 +4,5 @@
         <parent link="chassis"/>
         <child link="camera_link"/>
-        <origin xyz="0.257 0 1.165" rpy="0 0.610865 0"/>
+        <origin xyz="0.9 0 1.165" rpy="0 ${pi/2} 0"/>
     </joint>
     <link name="camera_link">

File: retos_ws/src/simulador_gazebo/models/Cybercrex_figuras/depth_camera.xacro (robot description, xacro)
@@ -4,12 +4,12 @@
         <parent link="chassis"/>
         <child link="camera_link"/>
-        <origin xyz="0.257 0 1.165" rpy="0 0.610865 0"/>
+        <origin xyz="0.305 0 0.08" rpy="0 0 0"/>
     </joint>
     <link name="camera_link">
         <visual>
             <geometry>
-                <box size="0.001 0.03 0.03"/>
+                <box size="0.010 0.03 0.03"/>
             </geometry>
-            <material name="black"/>
+            <material name="red"/>
         </visual>
     </link>
@@ -21,6 +21,6 @@
     <link name="camera_link_optical"></link>
     <gazebo reference="camera_link">
-        <material>Gazebo/Black</material>
-        <sensor name="camera" type="camera">
+        <material>Gazebo/Red</material>
+        <sensor name="camera" type="depth">
             <pose> 0 0 0 0 0 0 </pose>
             <visualize>true</visualize>
@@ -29,5 +29,5 @@
                 <horizontal_fov>1.089</horizontal_fov>
                 <image>
-                    <format>R8G8B8</format>
+                    <format>B8G8R8</format>
                     <width>640</width>
                     <height>480</height>
@@ -40,4 +40,6 @@
             <plugin name="camera_controller" filename="libgazebo_ros_camera.so">
                 <frame_name>camera_link_optical</frame_name>
+                <min_depth>0.1</min_depth>
+                <max_depth>100.0</max_depth>
             </plugin>
         </sensor>
